File: Design/uBike.brd (EAGLE design)
At the start: 55 x 85 mm, 101 parts, among them J10 455-1750-1-ND, J5 C167321, J6 C111196, J9 CONN_08, Q1 B772, Q2 B772, U1 RA-02_LORA, U10 MAX17048, U2 RP2040, U3 W25QXX128MBIT, U4 TMP102, U5 PAM2401, U6 AMS1117-3.3, U8 MCP73831, U9 LSM6DS0, Y1 12MHz

Commit message: New branch replacing Accel & Temp IC with pre-assembled module.
Parts:
- removed ADDR1: JUMPER-SMT_3_1-NC_TRACE_SILK, SparkFun-Jumpers:SMT-JUMPER_3_1-NC_TRACE_SILK
- removed C18: 10nF, rcl:C0402
- removed C21, C22: 0.1uF, rcl:C0402
- removed I2C_PU1: S_MODE, SparkFun-Jumpers:SMT-JUMPER_3_2-NC_TRACE_SILK
- removed JP3: ADD0, SparkFun-Passives:PAD-JUMPER-2-NC_BY_TRACE_YES_SILK
- removed L2: 30Ω, SparkFun-Coils:0603
- removed R17, R26: 4.7k, rcl:R0402
- removed R27: 10k, rcl:R0402
- removed R28: 100k, rcl:R0402
- removed R29: 10K, rcl:R0402
- removed SDX, SDX1: JUMPER-SMT_2_NC_TRACE_SILK, SparkFun-Jumpers:SMT-JUMPER_2_NC_TRACE_SILK
- removed U4: TMP102, SparkFun-Sensors:SOT563
- removed U9: LSM6DS0, temp:LGA14L
- added J14: (no value), SparkFun-Connectors:1X04
- moved U$30 26.1 mm to (42.9, 30.0), turned to 0 degrees
Connections:
- removed net !CS!: R27.1, U9.12
- removed net ADD0: R29.2, U4.4
- removed net INT1: U9.4
- removed net INT2: U9.9
- removed net N$15: JP3.1, R29.1
- removed net N$19: I2C_PU1.1, R17.2
- removed net N$20: I2C_PU1.3, R26.2
- removed net N$21: ADDR1.3, R28.1
- removed net OCS: U9.10
- removed net SCX: SDX.2, U9.3
- removed net SDI_AUX: SDX1.2, U9.2
- removed net SDO/SA0: ADDR1.2, U9.1
- removed net SDO_AUX: U9.11
- removed net VDD1: C21.1, L2.2, U9.8
- net 3.3V: now also J14.1; no longer C18.1, C22.1, I2C_PU1.2, L2.1, R27.2, R28.2, U4.5, U9.5
- net GND: now also J14.2; no longer ADDR1.1, C18.2, C21.2, C22.2, JP3.2, SDX.1, SDX1.1, U4.2, U9.6, U9.7
- net SCL: now also J14.3; no longer R17.1, U4.1, U9.13
- net SDA: now also J14.4; no longer R26.1, U4.6, U9.14
Routing:
- net 3.3V: track 334.4 -> 290.8 mm, vias 16 -> 13
- net SDA: track 96.6 -> 58.8 mm, vias 7 -> 5
- net SCL: track 92.1 -> 54.3 mm, vias 8 -> 5
- net N$20: track 16.4 -> 0.00 mm, vias 1 -> 0
- net SDO/SA0: track 12.9 -> 0.00 mm, vias 1 -> 0
- net N$19: track 11.6 -> 0.00 mm, vias 1 -> 0
- net SCX: track 9.08 -> 0.00 mm, vias 1 -> 0
- net SDI_AUX: track 8.42 -> 0.00 mm, vias 1 -> 0
- net N$15: track 7.25 -> 0.00 mm, vias 1 -> 0
- net N$21: track 6.45 -> 0.00 mm, vias 1 -> 0
- net VDD1: track 3.77 -> 0.00 mm
- net GND: track 28.2 -> 24.7 mm, vias 39 -> 37
- net ADD0: track 3.31 -> 0.00 mm
- net !CS!: track 2.72 -> 0.00 mm
- net GPIO3: track 44.9 -> 47.4 mm
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Other:
- board text removed: "X"
- board text removed: "Y"
- board text removed: "Z"

Commit message: Fixed U3 component with W25Q128JVSIQ
Parts:
- C10, C17, C20, C3, C4, C5, C6, C7, C8, C9: value 0.1uF -> 100nF
- H1, H2, H3, H4: value MOUNT-PAD-ROUND3.0 -> MOUNT-PAD-ROUND; device holes:3,0-PAD -> SpaceDIY_connectors:3,0-PAD
- R1: value 1.5 -> 1
- R25: value 2.0k -> 2k
- U3: value W25QXX128MBIT -> W25Q128JVSIQ; device SparkFun-IC-Memory:WSON-8-6X5-SKINNY_CENTERPAD -> SamacSys_Parts:SOIC127P790X216-8N
- moved U3 1.29 mm to (40.9, 39.8)
Connections:
- net GND: now also H1.P$2, H1.P$3, H1.P$4, H1.P$5, H1.P$6, H1.P$7, H1.P$8, H1.P$9, H2.P$2, H2.P$3, H2.P$4, H2.P$5, H2.P$6, H2.P$7, H2.P$8, H2.P$9, H3.P$2, H3.P$3, H3.P$4, H3.P$5, H3.P$6, H3.P$7, H3.P$8, H3.P$9, H4.P$2, H4.P$3, H4.P$4, H4.P$5, H4.P$6, H4.P$7, H4.P$8, H4.P$9
Routing:
- net 3.3V: track 290.8 -> 287.9 mm
- net QSPI-CS: track 15.7 -> 18.4 mm, vias 2 -> 4
- net QSPI-1: track 17.8 -> 19.2 mm
- net GND: track 24.7 -> 23.5 mm, vias 37 -> 36
- net QSPI-CLK: track 11.7 -> 12.2 mm
- net QSPI-3: track 20.3 -> 20.8 mm
- net QSPI-0: track 9.60 -> 10.1 mm
